File: hardware/10p-battery-holder/10p-battery-holder.kicad_pcb (KiCad board)
At the start: 2 copper layers, 225 x 80 mm, 14 parts, among them J1 Screw_Terminal_01x01, J10 Screw_Terminal_01x01, J2 Screw_Terminal_01x01, J3 Conn_01x02, J4 dual_18650_battery_holder, J5 dual_18650_battery_holder, J6 dual_18650_battery_holder, J7 dual_18650_battery_holder, J8 dual_18650_battery_holder, J9 Screw_Terminal_01x01

Commit message: Finished battery holder board!
Parts:
- moved J4 1.00 mm to (71.5, 90.5)
- moved J5 1.00 mm to (112.0, 90.5)
- moved J6 1.00 mm to (152.5, 90.5)
- moved J7 1.00 mm to (193.0, 90.5)
- moved J8 1.00 mm to (233.5, 90.5)
Connections:
- net Net-(J1-Pin_1) renamed /CELL+
- net Net-(J10-Pin_1) renamed /CELL-
Routing:
- net unconnected-(J3-MountPin-PadMP): track 0.00 -> 6.35 mm
- net /CELL-: track 0.00 -> 1.12 mm, vias 0 -> 817
- net /CELL+: track 0.00 -> 1.12 mm, vias 0 -> 819
- added copper zone on B.Cu, net /CELL+
- added copper zone on F.Cu, net /CELL+
- added copper zone on B.Cu, net /CELL-
- added copper zone on F.Cu, net /CELL-
Other:
- board text added: "+"
- board text added: "-"
- board text added: "CELL+"
- board text added: "CELL-"
- board text added: "CELL-TAPS"
- board text added: "Mark Belbin - 2023"
- board text added: "eSUP - 1S10P 18650 BATTERY BOARD"
