File: hardware/10p-battery-holder/10p-battery-holder.kicad_sch (KiCad schematic)
At the start: 14 parts, among them J1 Screw_Terminal_01x01, J4 dual_18650_battery_holder, J5 dual_18650_battery_holder, J6 Conn_01x02, J6 dual_18650_battery_holder, J7 dual_18650_battery_holder, J8 dual_18650_battery_holder

Commit message: Finished battery holder board!
Connections:
- net CELL+: now reaches J1.1 (Pin_1), J1.1 (Pin_1), J4.1 (CELL1+), J4.2 (CELL2+), J5.1 (CELL1+), J5.2 (CELL2+), J6.1 (CELL1+), J6.2 (CELL2+), J6.2 (Pin_2), J7.1 (CELL1+), J7.2 (CELL2+), J8.1 (CELL1+), J8.2 (CELL2+)
- net CELL-: now reaches J1.1 (Pin_1), J1.1 (Pin_1), J4.3 (CELL1-), J4.4 (CELL2-), J5.3 (CELL1-), J5.4 (CELL2-), J6.1 (Pin_1), J6.3 (CELL1-), J6.4 (CELL2-), J7.3 (CELL1-), J7.4 (CELL2-), J8.3 (CELL1-), J8.4 (CELL2-)
Other:
- moved on the sheet: J1
Changed lines of the file:
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@@
     (stroke (width 0) (type default))
   )
-  (wire (pts (xy 82.55 66.04) (xy 104.14 66.04))
+  (wire (pts (xy 90.17 66.04) (xy 104.14 66.04))
     (stroke (width 0) (type default))
   )
@@
     (stroke (width 0) (type default))
   )
-  (wire (pts (xy 82.55 105.41) (xy 104.14 105.41))
+  (wire (pts (xy 90.17 105.41) (xy 104.14 105.41))
     (stroke (width 0) (type default))
   )
@@
     (stroke (width 0) (type default))
   )
-  (text "CELL+" (at 63.5 67.31 0)
+  (text "CELL+" (at 71.12 67.31 0)
     (effects (font (size 1.27 1.27) (thickness 0.254) bold) (justify left bottom))
   )
@@
     (effects (font (size 1.016 1.016) italic) (justify left bottom))
   )
-  (text "CELL-" (at 62.23 105.41 0)
-    (effects (font (size 1.27 1.27) (thickness 0.254) bold) (justify left bottom))
-  )
-  (text "M4 Terminal\n" (at 63.5 69.85 0)
-    (effects (font (size 1.016 1.016) italic) (justify left bottom))
-  )
-  (text "M4 Terminal\n" (at 62.23 107.95 0)
+  (text "CELL-" (at 69.85 105.41 0)
+    (effects (font (size 1.27 1.27) (thickness 0.254) bold) (justify left bottom))
+  )
+  (text "M4 Terminal\n" (at 71.12 69.85 0)
+    (effects (font (size 1.016 1.016) italic) (justify left bottom))
+  )
+  (text "M4 Terminal\n" (at 69.85 107.95 0)
     (effects (font (size 1.016 1.016) italic) (justify left bottom))
   )
@@
     (effects (font (size 1.27 1.27) (thickness 0.254) bold) (justify left bottom))
   )
-  (symbol (lib_id "Connector:Screw_Terminal_01x01") (at 77.47 66.04 180) (unit 1)
-    (in_bom yes) (on_board yes) (dnp no)
-    (property "Reference" "J1" (at 73.66 66.04 0)
+  (label "CELL+" (at 92.71 66.04 0) (fields_autoplaced)
+    (effects (font (size 1.27 1.27)) (justify left bottom))
+  )
+  (label "CELL-" (at 92.71 105.41 0) (fields_autoplaced)
+    (effects (font (size 1.27 1.27)) (justify left bottom))
+  )
+  (symbol (lib_id "Connector:Screw_Terminal_01x01") (at 85.09 66.04 180) (unit 1)
+    (in_bom yes) (on_board yes) (dnp no)
+    (property "Reference" "J1" (at 81.28 66.04 0)
       (effects (font (size 1.27 1.27)))
     )
-    (property "Value" "Screw_Terminal_01x01" (at 75.438 64.7954 0)
-      (effects (font (size 1.27 1.27)) (justify left) hide)
-    )
-    (property "Footprint" "battery_holder:Wurth_746600430R" (at 77.47 66.04 0)
-      (effects (font (size 1.27 1.27)) hide)
-    )
-    (property "Datasheet" "~" (at 77.47 66.04 0)
-      (effects (font (size 1.27 1.27)) hide)
-    )
-    (property "MFG" "Würth Elektronik" (at 77.47 66.04 0)
-      (effects (font (size 1.27 1.27)) hide)
-    )
-    (property "MFG PN" "746600430R" (at 77.47 66.04 0)
+    (property "Value" "Screw_Terminal_01x01" (at 83.058 64.7954 0)
+      (effects (font (size 1.27 1.27)) (justify left) hide)
+    )
+    (property "Footprint" "battery_holder:Wurth_746600430R" (at 85.09 66.04 0)
+      (effects (font (size 1.27 1.27)) hide)
+    )
+    (property "Datasheet" "~" (at 85.09 66.04 0)
+      (effects (font (size 1.27 1.27)) hide)
+    )
+    (property "MFG" "Würth Elektronik" (at 85.09 66.04 0)
+      (effects (font (size 1.27 1.27)) hide)
+    )
+    (property "MFG PN" "746600430R" (at 85.09 66.04 0)
       (effects (font (size 1.27 1.27)) hide)
     )
@@
     )
   )
-  (symbol (lib_id "Connector:Screw_Terminal_01x01") (at 77.47 105.41 180) (unit 1)
-    (in_bom yes) (on_board yes) (dnp no)
-    (property "Reference" "J1" (at 73.66 105.41 0)
+  (symbol (lib_id "Connector:Screw_Terminal_01x01") (at 85.09 105.41 180) (unit 1)
+    (in_bom yes) (on_board yes) (dnp no)
+    (property "Reference" "J1" (at 81.28 105.41 0)
       (effects (font (size 1.27 1.27)))
     )
-    (property "Value" "Screw_Terminal_01x01" (at 75.438 104.1654 0)
-      (effects (font (size 1.27 1.27)) (justify left) hide)
-    )
-    (property "Footprint" "battery_holder:Wurth_746600430R" (at 77.47 105.41 0)
-      (effects (font (size 1.27 1.27)) hide)
-    )
-    (property "Datasheet" "~" (at 77.47 105.41 0)
-      (effects (font (size 1.27 1.27)) hide)
-    )
-    (property "MFG" "Würth Elektronik" (at 77.47 105.41 0)
-      (effects (font (size 1.27 1.27)) hide)
-    )
-    (property "MFG PN" "746600430R" (at 77.47 105.41 0)
-      (effects (font (size 1.27 1.27)) hide)
-    )
+    (property "Value" "Screw_Terminal_01x01" (at 83.058 104.1654 0)
+      (effects (font (size 1.27 1.27)) (justify left) hide)
+    )
+    (property "Footprint" "battery_holder:Wurth_746600430R" (at 85.09 105.41 0)
+      (effects (font (size 1.27 1.27)) hide)
+    )
+    (property "Datasheet" "~" (at 85.09 105.41 0)
+      (effects (font (size 1.27 1.27)) hide)
+    )
+    (property "MFG" "Würth Elektronik" (at 85.09 105.41 0)
+      (effects (font (size 1.27 1.27)) hide)
+    )
+    (property "MFG PN" "746600430R" (at 85.09 105.41 0)
+      (effects (font (size 1.27 1.27)) hide)
+    )
