File: hardware/10p-battery-board/10p-battery-holder.kicad_pcb (KiCad board)
At the start: 2 copper layers, 225 x 80 mm, 14 parts, among them J1 Screw_Terminal_01x01, J10 Screw_Terminal_01x01, J2 Screw_Terminal_01x01, J3 Conn_01x02, J4 dual_18650_battery_holder, J5 dual_18650_battery_holder, J6 dual_18650_battery_holder, J7 dual_18650_battery_holder, J8 dual_18650_battery_holder, J9 Screw_Terminal_01x01

Commit message: Exported gerbers for both boards
Changed lines of the file:
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@@
       (plot_on_all_layers_selection 0x0000000_00000000)
       (disableapertmacros false)
-      (usegerberextensions false)
-      (usegerberattributes true)
-      (usegerberadvancedattributes true)
-      (creategerberjobfile true)
+      (usegerberextensions true)
+      (usegerberattributes false)
+      (usegerberadvancedattributes false)
+      (creategerberjobfile false)
       (dashed_line_dash_ratio 12.000000)
       (dashed_line_gap_ratio 3.000000)
@@
       (psa4output false)
       (plotreference true)
-      (plotvalue true)
+      (plotvalue false)
       (plotinvisibletext false)
       (sketchpadsonfab false)
-      (subtractmaskfromsilk false)
+      (subtractmaskfromsilk true)
       (outputformat 1)
       (mirror false)
-      (drillshape 1)
+      (drillshape 0)
       (scaleselection 1)
-      (outputdirectory "")
+      (outputdirectory "gerbers/")
     )
   )
@@
     (pad "2" smd roundrect (at 0.625 -2.4 90) (size 0.8 1.6) (layers "F.Cu" "F.Paste" "F.Mask") (roundrect_rratio 0.25)
       (net 6 "/CELL+") (pinfunction "Pin_2") (pintype "passive"))
-    (pad "MP" smd roundrect (at -3.175 0.5 90) (size 2.1 3) (layers "F.Cu" "F.Paste" "F.Mask") (roundrect_rratio 0.119048)
+    (pad "MP" smd roundrect (at -3.175 0.5 90) (size 2.1 3) (layers "F.Cu" "F.Paste" "F.Mask") (roundrect_rratio 0.1190480952)
       (net 5 "unconnected-(J3-MountPin-PadMP)") (pinfunction "MountPin") (pintype "passive+no_connect"))
-    (pad "MP" smd roundrect (at 3.175 0.5 90) (size 2.1 3) (layers "F.Cu" "F.Paste" "F.Mask") (roundrect_rratio 0.119048)
+    (pad "MP" smd roundrect (at 3.175 0.5 90) (size 2.1 3) (layers "F.Cu" "F.Paste" "F.Mask") (roundrect_rratio 0.1190480952)
       (net 5 "unconnected-(J3-MountPin-PadMP)") (pinfunction "MountPin") (pintype "passive+no_connect"))
     (model "${KICAD6_3DMODEL_DIR}/Connector_Molex.3dshapes/Molex_PicoBlade_53261-0271_1x02-1MP_P1.25mm_Horizontal.wrl"
@@
     (pts (xy 40 130.5) (xy 265 130.5))
     (height 4.999999)
-    (gr_text "225.0000 mm" (at 152.5 134.349999) (layer "F.Fab")
+    (gr_text "8858.2677 mils" (at 152.5 134.349999) (layer "F.Fab")
       (effects (font (size 1 1) (thickness 0.15)))
     )
@@
     (pts (xy 265 130.5) (xy 265 50.5))
     (height 10)
-    (gr_text "80.0000 mm" (at 273.85 90.5 90) (layer "F.Fab")
+    (gr_text "3149.6063 mils" (at 273.85 90.5 90) (layer "F.Fab")
       (effects (font (size 1 1) (thickness 0.15)))
     )
